File: KiCAD_files/Feeder.kicad_sch (KiCad schematic)
At the start: 82 parts, among them J405 Conn_01x02_Male, J406 Conn_01x02_Male, J501 Conn_01x03, Q501 60V N channel, Q502 TK13P25D,RQ, T501 PA2467NL, U407 OPA316, U501 NCP12700, U503 TL431MFDT,215, U505 MCP1799T-5002H/DB

Commit message: corrected version number in template
Other:
- title: OWNVERTER V1.1 -> OWNVERTER V1.0
Changed lines of the file:
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@@
   (paper "A3")
   (title_block
-    (title "OWNVERTER V1.1")
+    (title "OWNVERTER V1.0")
     (comment 1 "TWR")
   )
