File: KiCAD_files/High_side.kicad_sch (KiCad schematic)
At the start: 27 parts

Commit message: corrected version number in template
Other:
- title: OWNVERTER V1.1 -> OWNVERTER V1.0
Changed lines of the file:
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@@
   (paper "A3")
   (title_block
-    (title "OWNVERTER V1.1")
+    (title "OWNVERTER V1.0")
     (comment 1 "TWR")
   )
