File: KiCAD_files/InverterLeg.kicad_sch (KiCad schematic)
At the start: 76 parts, among them Q699 DMP3099L-7, U601 AMC1100DUB, U603 UCC21222DR, U605 ACS730KLCTR-20AB

Commit message: corrected version number in template
Other:
- title: OWNVERTER V1.1 -> OWNVERTER V1.0
Changed lines of the file:
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@@
   (paper "A3")
   (title_block
-    (title "OWNVERTER V1.1")
+    (title "OWNVERTER V1.0")
     (comment 1 "TWR")
   )
