File: KiCAD_files/Microcontroller.kicad_sch (KiCad schematic)
At the start: 79 parts, among them J403 RJ45_LED_Shielded, J404 RJ45_LED_Shielded, J801 Conn_01x04, U401 OwnTech_SPIN, U402 TCAN334GDR, U405 LTC2850xS8, U406 OPA2277, U410 TS5A3357DCUT

Commit message: corrected version number in template
Other:
- title: OWNVERTER V1.1 -> OWNVERTER V1.0
Changed lines of the file:
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@@
   (paper "A3")
   (title_block
-    (title "OWNVERTER V1.1")
+    (title "OWNVERTER V1.0")
     (company "https://gitlab.laas.fr/owntech/1leg/-/tree/V1.1.2/KiCAD_files")
     (comment 1 "TWR")
