File: KiCAD_files/Microcontroller.kicad_sch (KiCad schematic)
At the start: 79 parts, among them J403 RJ45_LED_Shielded, J404 RJ45_LED_Shielded, J801 Conn_01x04, U401 OwnTech_SPIN, U402 TCAN334GDR, U405 LTC2850xS8, U406 OPA2277, U410 TS5A3357DCUT

Commit message: Added ERC rules for galvanic isolation. Modified SPIN pinout.
Signed-off-by: Jean Alinei <jean.alinei@laas.fr>
Parts:
- renumbered J801 to J301
Other:
- moved on the sheet: C410, D403, JP403, JP408, JP409, JP417, R402, R403, R404, R405, R409, R410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
